Commit message: Added image capturer

File: ur5_gripper_moveit_config/config/gazebo_ur5 (copy).urdf (robot description, URDF)
Before this commit: robot ur5, 23 links, 22 joints
Links:
- added link camera_link_1, mass 0.2; collision box size=0.008 0.13 0.02; visual mesh filename=package://ur5_visual_servos/meshes/intel_realsense_r200/mes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 scale=1 1 1
- added link camera_link_2, mass 0.2; collision box size=0.008 0.13 0.02; visual mesh filename=package://ur5_visual_servos/meshes/intel_realsense_r200/mes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 scale=1 1 1
Joints:
- added joint camera_joint_1: type fixed, parent world, child camera_link_1, origin xyz=0.25 1.2 0.4 rpy=0 0 -1.57, axis 0 1 0
- added joint camera_joint_2: type fixed, parent world, child camera_link_2, origin xyz=-0.4 1.2 0.4 rpy=0 0 -1.047, axis 0 1 0

File: ur5_gripper_moveit_config/config/gazebo_ur5.urdf (robot description, URDF)
Before this commit: robot ur5, 25 links, 24 joints
Links:
- added link gripper_indicator_link; visual sphere radius=0.06
Joints:
- added joint gripper_indicator_joint: type fixed, parent robotiq_85_base_link, child gripper_indicator_link, origin xyz=0 0 0 rpy=0 0 0
