Commit message: Added needle tool, Jacobian updater

File: ur5_gripper_moveit_config/config/gazebo_ur5.urdf (robot description, URDF)
Before this commit: robot ur5, 26 links, 25 joints
Links:
- added link frame_tool_link; visual cylinder length=0.15 radius=0.01
- added link needle_tool_link; visual cylinder length=0.2 radius=0.01
- link robotiq_85_left_finger_link: geometry collision mesh filename=package://robotiq_description/meshes/collision/robotiq_85_f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
- link robotiq_85_left_finger_tip_link: geometry collision mesh filename=package://robotiq_description/meshes/collision/robotiq_85_f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
- link robotiq_85_left_inner_knuckle_link: geometry collision mesh filename=package://robotiq_description/meshes/collision/robotiq_85_i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
- link robotiq_85_left_knuckle_link: geometry collision mesh filename=package://robotiq_description/meshes/collision/robotiq_85_k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
- link robotiq_85_right_finger_link: geometry collision mesh filename=package://robotiq_description/meshes/collision/robotiq_85_f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
- link robotiq_85_right_finger_tip_link: geometry collision mesh filename=package://robotiq_description/meshes/collision/robotiq_85_f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
- link robotiq_85_right_inner_knuckle_link: geometry collision mesh filename=package://robotiq_description/meshes/collision/robotiq_85_i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
- link robotiq_85_right_knuckle_link: geometry collision mesh filename=package://robotiq_description/meshes/collision/robotiq_85_k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
Joints:
- added joint frame_tool_joint: type fixed, parent robotiq_85_base_link, child frame_tool_link, origin xyz=0 0.075 0 rpy=1.57 0 0
- added joint needle_tool_joint: type fixed, parent robotiq_85_base_link, child needle_tool_link, origin xyz=0.1 0 0 rpy=0 1.57 0

Commit message: Added J updater

File: ur5_gripper_moveit_config/config/gazebo_ur5.urdf (robot description, URDF)
Before this commit: robot ur5, 28 links, 27 joints
Links:
- removed link gripper_indicator_link
- added link needle_tip_link; visual sphere radius=0.01
Joints:
- removed joint gripper_indicator_joint
- added joint needle_tip_joint: type fixed, parent robotiq_85_base_link, child needle_tip_link, origin xyz=0.21 0 0 rpy=0 1.57 0

Commit message: Updated position servo

File: ur5_gripper_moveit_config/config/gazebo_ur5.urdf (robot description, URDF)
Before this commit: robot ur5, 28 links, 27 joints
Links:
- added link frame_tip_link; visual sphere radius=0.005
- added link gripper_indicator_link; visual sphere radius=0.01
- link frame_tool_link: geometry visual cylinder length=0.15 radius=0.005
- link needle_tip_link: geometry visual sphere radius=0.005
- link needle_tool_link: geometry visual cylinder length=0.2 radius=0.005
- link robotiq_85_base_link: geometry collision mesh filename=package://robotiq_description/meshes/collision/robotiq_85_b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
- link robotiq_coupler: geometry collision mesh filename=package://robotiq_description/meshes/robotiq_85_coupler.stl
Joints:
- added joint frame_tip_joint: type fixed, parent robotiq_85_base_link, child frame_tip_link, origin xyz=0 0.155 0 rpy=1.57 0 0
- added joint gripper_indicator_joint: type fixed, parent robotiq_85_base_link, child gripper_indicator_link, origin xyz=0 0 0 rpy=0 0 0
- joint needle_tip_joint: origin xyz=0.21 0 0 rpy=0 1.57 0 -> xyz=0.205 0 0 rpy=0 1.57 0

Commit message: Working version of orientation servo w/ separate stages

File: ur5_gripper_moveit_config/config/gazebo_ur5.urdf (robot description, URDF)
Before this commit: robot ur5, 30 links, 29 joints
Links:
- link wrist_3_link: geometry collision mesh filename=package://ur_description/meshes/ur5/collision/wrist3.stl
Joints:
- joint camera_joint_1: origin xyz=0.25 1.2 0.4 rpy=0 0 -1.57 -> xyz=0.75 1.0 0.4 rpy=0 0 -1.96
- joint camera_joint_2: origin xyz=-0.4 1.2 0.4 rpy=0 0 -1.047 -> xyz=-0.4 0.6 0.4 rpy=0 0 -0.523
