Commit message: Organized directories

File: Gazebo_ROS_Simulations/ur5_gripper_moveit_config/config/gazebo_ur5.urdf (robot description, URDF)
Before this commit: robot ur5, 30 links, 29 joints
Links:
- removed link frame_tip_link
- removed link frame_tool_link
- removed link gripper_indicator_link
- removed link needle_tip_link
- removed link needle_tool_link
Joints:
- removed joint frame_tip_joint
- removed joint frame_tool_joint
- removed joint gripper_indicator_joint
- removed joint needle_tip_joint
- removed joint needle_tool_joint
